File: IEEE-Clock-Charlie/IEEE-Clock-Charlie.kicad_pcb (KiCad board)
At the start: 2 copper layers, 189.9 x 38.1 mm, 12 parts, among them M1 MountingHole_3.2mm_M3, M2 MountingHole_3.2mm_M3, M3 MountingHole_3.2mm_M3, M4 MountingHole_3.2mm_M3, U1 ADA_CHARLIE, U2 ADA_CHARLIE, U3 ADA_CHARLIE, U4 ADA_DS3231

Commit message: With jumpers routed and ready to go
Parts:
- added A1: SolderJumper_2_Open, Jumper:SolderJumper-2_P1.3mm_Open_RoundedPad1.0x1.5mm, B.Cu at (125.5, 109.5)
- added A2: SolderJumper_2_Open, Jumper:SolderJumper-2_P1.3mm_Open_RoundedPad1.0x1.5mm, B.Cu at (118.4, 109.5)
- added A3: SolderJumper_2_Open, Jumper:SolderJumper-2_P1.3mm_Open_RoundedPad1.0x1.5mm, B.Cu at (111.5, 109.2)
- added C1: SolderJumper_2_Open, Jumper:SolderJumper-2_P1.3mm_Open_RoundedPad1.0x1.5mm, B.Cu at (125.5, 105.2)
- added C2: SolderJumper_2_Open, Jumper:SolderJumper-2_P1.3mm_Open_RoundedPad1.0x1.5mm, B.Cu at (118.4, 104.9)
- added C3: SolderJumper_2_Open, Jumper:SolderJumper-2_P1.3mm_Open_RoundedPad1.0x1.5mm, B.Cu at (111.5, 105.2)
- added D1: SolderJumper_2_Open, Jumper:SolderJumper-2_P1.3mm_Open_RoundedPad1.0x1.5mm, B.Cu at (125.4, 100.8)
- added D2: SolderJumper_2_Open, Jumper:SolderJumper-2_P1.3mm_Open_RoundedPad1.0x1.5mm, B.Cu at (118.4, 100.8)
- added D3: SolderJumper_2_Open, Jumper:SolderJumper-2_P1.3mm_Open_RoundedPad1.0x1.5mm, B.Cu at (111.5, 100.8)
- U4: footprint IEEE-Clock-Charlie:ADA_DS3231_MOD -> Connector_PinHeader_2.54mm:PinHeader_1x08_P2.54mm_Vertical
- renumbered A1 to N1
Connections:
- N1 pad 13: Net-(A1-Pad13) -> Net-(C1-Pad1)
- N1 pad 23: Net-(A1-Pad23) -> Net-(A1-Pad2)
- N1 pad 24: Net-(A1-Pad24) -> Net-(A2-Pad2)
- N1 pad 6: Net-(A1-Pad6) -> Net-(D1-Pad1)
- N1 pad 7: Net-(A1-Pad7) -> Net-(D2-Pad1)
- N1 pad 8: Net-(A1-Pad8) -> Net-(D3-Pad1)
- U1 pad 16: Net-(A1-Pad24) -> Net-(C1-Pad1)
- U1 pad 17: Net-(A1-Pad23) -> Net-(D1-Pad1)
- U1 pad 2: Net-(A1-Pad23) -> Net-(A1-Pad1)
- U2 pad 16: Net-(A1-Pad24) -> Net-(C1-Pad1)
- U2 pad 17: Net-(A1-Pad23) -> Net-(D2-Pad1)
- U2 pad 2: Net-(A1-Pad24) -> Net-(A2-Pad1)
- U3 pad 16: Net-(A1-Pad24) -> Net-(C1-Pad1)
- U3 pad 17: Net-(A1-Pad23) -> Net-(D3-Pad1)
- U3 pad 2: GND -> Net-(A3-Pad1)
- U4 pad 3: Net-(A1-Pad24) -> Net-(A2-Pad2)
- U4 pad 4: Net-(A1-Pad23) -> Net-(A1-Pad2)
Routing:
- net Net-(A1-Pad23): track 157.4 -> 0.00 mm
- net Net-(C1-Pad1): track 0.00 -> 144.5 mm
- net Net-(A1-Pad24): track 131.1 -> 0.00 mm
- net Net-(D1-Pad1): track 0.00 -> 93.8 mm, vias 0 -> 1
- net Net-(A1-Pad1): track 0.00 -> 70.9 mm
- net Net-(A1-Pad2): track 0.00 -> 70.5 mm, vias 0 -> 1
- net Net-(A2-Pad2): track 0.00 -> 66.2 mm, vias 0 -> 1
- net Net-(D3-Pad1): track 0.00 -> 62.3 mm, vias 0 -> 1
- net Net-(D2-Pad1): track 0.00 -> 61.5 mm, vias 0 -> 1
- net Net-(A2-Pad1): track 0.00 -> 33.7 mm
- net Net-(L1-Pad1): track 71.8 -> 96.6 mm
- net Net-(N1-Pad10): track 96.4 -> 117.5 mm
- net Net-(N1-Pad12): track 82.1 -> 94.1 mm
- net Net-(A3-Pad1): track 0.00 -> 7.82 mm
- net Net-(N1-Pad11): track 80.5 -> 82.9 mm
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